File: BPEM488TDHAux.sch (KiCad schematic (older format))
At the start: 100 parts, among them J1 Conn_01x02, J2 Conn_02x18_Odd_Even, J3 DB15_Female, J4 DB15_Female, Q1 ZTX450, Q10 ZTX450, Q11 ZTX450, Q12 ZTX450, Q13 ZTX450, Q14 ZTX450, Q15 ZTX450, Q16 ZTX450, Q17 ZTX450, Q18 ZTX450, Q19 ZTX450, Q2 ZTX450, Q20 ZTX450, Q21 ZTX450, Q22 ZTX450, Q23 ZTX450, Q24 ZTX450, Q25 ZTX450, Q3 ZTX450, Q4 ZTX450, Q5 ZTX450, Q6 ZTX450, Q7 ZTX450, Q8 ZTX450, Q9 ZTX450, U1 LD1085V50, U2 L7808ABV

Commit message: Add files via upload
Parts:
- J2: footprint Connector_PinHeader_2.54mm:PinHeader_2x18_P2.54mm_Vertical -> Connector_PinSocket_2.54mm:PinSocket_2x18_P2.54mm_Vertical
- J3, J4: Digikey 609-1499-ND -> A32123-ND; Mfg D15S33E4GX00LF -> 5747845-6
Connections:
- net labels added: PA0
- net labels removed: PA2
- wire segments 362 -> 364
- no-connect marks 5 -> 3
Other:
- moved on the sheet: J2, J3, J4, Q1, Q10, Q11, Q12, Q13, Q14, Q15, Q16, Q17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

Commit message: Add files via upload
Connections:
- net labels added: +12V
- wire segments 364 -> 369

Commit message: Add files via upload
Other:
- note added: "PB0 = FP = Fuel Pump Relay\nPB1 - ASD = Automatic Shutdown Relay\nPB2 = Alarm = Audible Alarm Relay\nPB3 = AIOT = Accumulated Injector On Time Counter\nPB4 = PB4out = PB4 output spare\nPB5 = PB5out = PB5 output spare\nPB6 = PB6out = PB6 output spare\nPK0 = LOP = Low Oil Pressure Alarm\nPK1 = HOT = High Oil Pressure Alarm\nPK2 = HET = High Engine Temperature A;arm\nPK3 = HEGT = High Exhaust Temper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"
- note added: "PT3 = Ign1 = 1&6\nPT4 = Ign2 = 10&5\nPT5 = Ign3 = 9&8\nPT6 = Ign4 = 4&7\nPT7 = Ign5 = 3&2\nPP0 = Inj1 = 1&10\nPP1 = Inj2 = 9&4\nPP2 = Inj3 = 3&6\nPP3 = Inj4 = 5&8\nPP4 = Inj3 = 7&2"
- moved on the sheet: J2, J3, J4, Q1, Q10, Q11, Q12, Q13, Q14, Q15, Q16, Q17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

Commit message: Add files via upload
Parts:
- removed C2, C4, C5: 33uF, Capacitor_THT:CP_Radial_Tantal_D8.0mm_P5.00mm, symbol Device:CP1
- removed U1: LD1085V50, Package_TO_SOT_THT:TO-220-3_Horizontal_TabDown, symbol Regulator_Linear:LM7805_TO220
- removed U2: L7808ABV, Package_TO_SOT_THT:TO-220-3_Horizontal_TabDown, symbol Regulator_Linear:LM7808_TO220
- added C2, C4: 10uF, Capacitor_THT:C_Disc_D5.0mm_W2.5mm_P2.50mm, symbol Device:C
- added C5: 0.1uF, Capacitor_THT:C_Disc_D5.0mm_W2.5mm_P2.50mm, symbol Device:C
- added RV1: B72214S1140K501, Varistor:RV_Disc_D15.5mm_W3.9mm_P7.5mm, symbol Device:Varistor
- added U1: LD1085, Package_TO_SOT_THT:TO-220F-3_Horizontal_TabDown, symbol BPEM488TDHAux-rescue:LD1085-BPEM488TDHAux-cache
- added U2: LD7808, Package_TO_SOT_THT:TO-220F-3_Horizontal_TabDown, symbol BPEM488TDHAux-rescue:LD7808-BPEM488TDHAux-cache
- J1: value Conn_01x02 -> Molex 0026013114
- J3, J4: footprint digikey-footprints:DB15FC -> Connector_Dsub:DSUB-15_Female_Horizontal_P2.77x2.84mm_EdgePinOffset7.70mm_Housed_MountingHolesOffset9.12mm
Connections:
- wire segments 369 -> 374
Other:
- note added: "Insulate tab on U1!!!"
- moved on the sheet: J1
