File: BPEM488TDHAux.kicad_pcb (KiCad board)
At the start: 2 copper layers, 152.4 x 101.6 mm, 100 parts, among them J1 Conn_01x02, J2 Conn_02x18_Odd_Even, J3 DB15_Female, J4 DB15_Female, Q1 ZTX450, Q10 ZTX450, Q11 ZTX450, Q12 ZTX450, Q13 ZTX450, Q14 ZTX450, Q15 ZTX450, Q16 ZTX450, Q17 ZTX450, Q18 ZTX450, Q19 ZTX450, Q2 ZTX450, Q20 ZTX450, Q21 ZTX450, Q22 ZTX450, Q23 ZTX450, Q24 ZTX450, Q25 ZTX450, Q3 ZTX450, Q4 ZTX450, Q5 ZTX450, Q6 ZTX450, Q7 ZTX450, Q8 ZTX450, Q9 ZTX450, U1 LD1085V50, U2 L7808ABV

Commit message: Add files via upload
Parts:
- moved S1 41.7 mm to (55.9, 65.6), turned to 90 degrees
- moved Q21 41.0 mm to (185.4, 96.5)
- moved Q25 41.0 mm to (185.4, 55.9)
- moved R41 41.0 mm to (180.3, 96.5)
- moved R42 41.0 mm to (180.3, 101.6)
- moved R49 41.0 mm to (180.3, 55.9)
- moved R50 41.0 mm to (180.3, 61.0)
- moved J3 22.9 mm to (59.7, 99.0)
- moved R43 20.9 mm to (180.3, 86.4)
- moved R44 20.9 mm to (180.3, 91.4)
- moved R47 20.9 mm to (180.3, 66.0)
- moved R48 20.9 mm to (180.3, 71.1)
- moved Q22 20.9 mm to (185.4, 86.4)
- moved Q24 20.9 mm to (185.4, 66.0)
- moved S2 17.2 mm to (55.9, 137.2), turned to 90 degrees
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Connections:
- C1 pad 1: Net-(C1-Pad1) -> +BATT
- C2 pad 1: +BATT -> +12V
- C3 pad 1: +BATT -> +12V
- D1 pad 1: Net-(C1-Pad1) -> +BATT
- D3 pad 1: +BATT -> +12V
- D3 pad 2: Net-(C1-Pad1) -> +BATT
- D4 pad 1: +BATT -> +12V
- D5 pad 1: +BATT -> +12V
- D6 pad 1: +BATT -> +12V
- J1 pad 1: Net-(C1-Pad1) -> +BATT
- J2 pad 13: /PK5 -> GND
- J2 pad 15: /PK4 -> GND
- J2 pad 17: /PB0 -> GND
- J2 pad 19: /PB1 -> GND
- J2 pad 21: /PB2 -> VDD
- J2 pad 23: /PB3 -> +BATT
- J2 pad 25: /PB4 -> /RESET
- J2 pad 26: +8V -> /PK5
- J2 pad 27: /PB5 -> /PA0
- J2 pad 28: VDD -> /PK4
- J2 pad 29: /PB6 -> +8V
- J2 pad 30: GND -> /PB0
- J2 pad 31: /RESET -> /PB6
- J2 pad 32: GND -> /PB1
- J2 pad 33: +BATT -> /PB5
- J2 pad 34: /PA0 -> /PB2
- J2 pad 35: GND -> /PB4
- J2 pad 36: GND -> /PB3
- J3 pad 1: /FP -> /PB5out
- J3 pad 10: /AIOT -> /PB4out
- J3 pad 11: /PP5out -> /AIOT
- J3 pad 12: /HOT -> /Alarm
- J3 pad 13: /HEGT -> /ASD
- J3 pad 14: /LFP -> /FP
- J3 pad 15: /PB5out -> /LFP
- J3 pad 2: /Alarm -> /LOP
- J3 pad 3: /PB4out -> /HOT
- J3 pad 4: /LOP -> /HET
- J3 pad 5: /HET -> /HEGT
- J3 pad 6: /HFT -> /PP5out
- J3 pad 8: /PB6out -> /HFT
- J3 pad 9: /ASD -> /PB6out
- J4 pad 1: Net-(J4-Pad1) -> /Ign1
- J4 pad 10: /Ign3 -> /Ign2
- J4 pad 11: /Ign1 -> /Ign3
- J4 pad 12: /Inj5 -> /Ign4
- J4 pad 13: /Inj3 -> /Ign5
- J4 pad 14: /Inj1 -> Net-(J4-Pad14)
- J4 pad 15: +BATT -> VDD
- J4 pad 2: /Ign4 -> /Inj4
- J4 pad 3: /Ign2 -> /Inj3
- J4 pad 4: Net-(J4-Pad4) -> /Inj2
- J4 pad 5: /Inj4 -> /Inj1
- J4 pad 6: /Inj2 -> Net-(J4-Pad6)
- J4 pad 7: VDD -> Net-(J4-Pad7)
- J4 pad 8: Net-(J4-Pad8) -> +12V
- J4 pad 9: /Ign5 -> /Inj5
- U1 pad 1: +BATT -> +12V
- U2 pad 1: +BATT -> +12V
Routing:
- net /PA0: track 0.00 -> 179.5 mm
- net +12V: track 0.00 -> 172.9 mm, vias 0 -> 1
- net /RESET: track 0.00 -> 116.3 mm
- net +BATT: track 0.00 -> 112.2 mm
- net /PP0: track 0.00 -> 112.1 mm, vias 0 -> 1
- net VDD: track 0.00 -> 109.0 mm, vias 0 -> 1
- net /PP1: track 0.00 -> 97.9 mm, vias 0 -> 1
- net /PP3: track 0.00 -> 87.2 mm, vias 0 -> 1
- net +8V: track 0.00 -> 86.6 mm, vias 0 -> 1
- net /PP4: track 0.00 -> 85.9 mm, vias 0 -> 1
- net /PP2: track 0.00 -> 84.6 mm, vias 0 -> 1
- net /PK5: track 0.00 -> 82.7 mm
- net /PK4: track 0.00 -> 79.9 mm
- net /PB0: track 0.00 -> 73.0 mm
- net /PB1: track 0.00 -> 65.2 mm
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- added copper zone on B.Cu, net GND
- added copper zone on F.Cu, net GND
Other:
- net class 1 amp added: clearance 0.3, trace_width 0.3, via_dia 0.8, via_drill 0.4

Commit message: Add files via upload
Parts:
- added REF**: MountingHole_3mm_Pad, MountingHole:MountingHole_3mm_Pad, F.Cu at (163.3, 141.6)
- added RV1: B72214S1140K501, Varistor:RV_Disc_D15.5mm_W3.9mm_P7.5mm, F.Cu at (104.1, 143.6)
- C2, C4: value 33uF -> 10uF; footprint Capacitor_THT:CP_Radial_Tantal_D8.0mm_P5.00mm -> Capacitor_THT:C_Disc_D5.0mm_W2.5mm_P2.50mm
- C5: value 33uF -> 0.1uF; footprint Capacitor_THT:CP_Radial_Tantal_D8.0mm_P5.00mm -> Capacitor_THT:C_Disc_D5.0mm_W2.5mm_P2.50mm
- J1: value Conn_01x02 -> Molex 0026013114
- J3, J4: footprint digikey-footprints:DB15FC -> Connector_Dsub:DSUB-15_Female_Horizontal_P2.77x2.84mm_EdgePinOffset7.70mm_Housed_MountingHolesOffset9.12mm
- U1: value LD1085V50 -> LD1085; footprint Package_TO_SOT_THT:TO-220-3_Horizontal_TabDown -> Package_TO_SOT_THT:TO-220F-3_Horizontal_TabDown
- U2: value L7808ABV -> LD7808; footprint Package_TO_SOT_THT:TO-220-3_Horizontal_TabDown -> Package_TO_SOT_THT:TO-220F-3_Horizontal_TabDown
- moved C4 20.9 mm to (135.9, 137.2)
- moved J3 10.1 mm to (57.7, 109.0), turned to 270 degrees
- moved J4 10.1 mm to (196.2, 73.7), turned to 90 degrees
- moved D5 7.62 mm to (143.5, 133.3), turned to 180 degrees
- moved C5 6.82 mm to (188.4, 141.0), turned to 270 degrees
- moved C2 6.48 mm to (129.5, 134.6), turned to 0 degrees
- moved U1 2.29 mm to (136.5, 129.5)
- moved U2 2.22 mm to (173.4, 129.5)
Connections:
- J4 pad 8: +12V -> +BATT
- U1 pad 1: +12V -> GND
- U1 pad 2: GND -> Net-(C4-Pad1)
- U1 pad 3: Net-(C4-Pad1) -> +12V
Routing:
- net +BATT: track 112.2 -> 261.7 mm, vias 0 -> 2
- net +12V: track 172.9 -> 91.8 mm, vias 1 -> 0
- net Net-(C4-Pad1): track 21.5 -> 28.0 mm
- net /Ign1: track 46.5 -> 40.2 mm
- net /Inj5: track 27.8 -> 22.3 mm
- net /PB6out: track 34.4 -> 38.5 mm
- net /Ign2: track 35.7 -> 39.6 mm
- net /HET: track 31.8 -> 35.6 mm
- net /Alarm: track 11.6 -> 15.3 mm
- net /FP: track 25.3 -> 29.0 mm
- net /ASD: track 17.7 -> 21.4 mm
- net /Ign3: track 35.2 -> 38.8 mm
- net /Ign5: track 47.1 -> 50.8 mm
- net /PB4out: track 19.9 -> 23.5 mm
- net /AIOT: track 14.5 -> 18.1 mm
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Other:
- board text added: "BPEM488 Aux Designed by Robert Hiebert 7-18-20"
- board text added: "Insulate Tab"

Commit message: Add files via upload
Other:
- board text added: "5 Volt"
- board text added: "8 Volt"
- board text added: "EEEM Load"
- board text added: "Reset"
